Commit message: Checked sensors

File: sandwich_description/urdf/sandwich.xacro (robot description, xacro)
@@ -12,5 +12,5 @@
   <!-- Note: this is only used for some sensors that do not correctly use the
   robotNamespace parameter -->
-  <!-- <xacro:property name="namespace" value="$(arg namespace)" scope="global" /> -->
+  <xacro:property name="namespace" value="$(arg namespace)" scope="global" />
   <!-- Thrusters -->
   <xacro:arg name="thruster_namespace" default="thrusters/"/>
@@ -19,10 +19,10 @@
   <xacro:add_thrusters namespace="$(arg namespace)"/>
   <!-- Decide if we lock the robot to the world -->
-  <!-- <xacro:if value="$(arg locked)">
+  <xacro:if value="$(arg locked)">
     <gazebo>
-      <link name="sandwich_external_link"/>
-      <joint name="sandwich_external_pivot_joint" type="universal">
-        <parent>sandwich::sandwich/base_link</parent>
-        <child>sandwich_external_link</child>
+      <link name="$(arg namespace)/sandwich_external_link"/>
+      <joint name="$(arg namespace)/sandwich_external_pivot_joint" type="universal">
+        <parent>$(arg namespace)::$(arg namespace)/base_link</parent>
+        <child>$(arg namespace)/sandwich_external_link</child>
         <axis>
           <xyz>1 0 0</xyz>
@@ -32,7 +32,7 @@
         </axis2>
       </joint>
-      <joint name="sandwich_external_riser" type="prismatic">
+      <joint name="$(arg namespace)/sandwich_external_riser" type="prismatic">
         <parent>world</parent>
-        <child>sandwich_external_link</child>
+        <child>$(arg namespace)/sandwich_external_link</child>
         <axis>
           <limit>
@@ -44,7 +44,7 @@
       </joint>
     </gazebo>
-  </xacro:if> -->
+  </xacro:if>
   <!-- Sensors -->
- <!--  <xacro:arg name="camera_namespace" default="cameras/"/>
+  <xacro:arg name="camera_namespace" default="cameras/"/>
   <xacro:arg name="sensor_namespace" default="sensors/"/>
   <xacro:arg name="pinger_namespace" default="pingers/"/>
@@ -61,4 +61,4 @@
   	update_rate="20" />
   <xacro:wamv_imu name="imu" y="-0.2" z="1.0" update_rate="100" />
-  <xacro:wamv_pinger name="pinger" frameId="sandwich/pinger" /> -->
+  <xacro:wamv_pinger name="pinger" frameId="$(arg namespace)/pinger" />
 </robot>
