Commit message: Fixed thruster orientation and position

File: sandwich_description/urdf/thrusters.xacro (robot description, xacro)
@@ -4,4 +4,10 @@
     <!-- Dummy link, which usv_gazebo_thrust_plugin looks for -->
     <link name="left_engine_link">
+      <visual>
+        <origin rpy="0 0 -${pi/2}" xyz="0 0 0"/>
+        <geometry>
+          <mesh filename="package://sandwich_description/models/thruster/thruster.dae" scale="4 4 4"/>
+        </geometry>
+      </visual>
       <inertial>
         <mass value="0.1"/>
@@ -12,6 +18,7 @@
     <link name="left_propeller_link">
       <visual>
+         <origin rpy="0 0 -${pi/2}" xyz="0 0 0"/>
         <geometry>
-          <mesh filename="package://sandwich_description/models/propeller/propeller.dae"/>
+          <mesh filename="package://sandwich_description/models/propeller/propeller.dae" scale="4 4 4"/>
         </geometry>
       </visual>
@@ -23,6 +30,6 @@
     <!-- Dummy joint, which usv_gazebo_thrust_plugin looks for -->
     <joint name="left_chasis_engine_joint" type="revolute">
-      <axis xyz="0 0 1"/>
-      <origin rpy="0 0 0" xyz="-6.103 0.911 0.016"/>
+      <axis xyz="1 0 0"/>
+      <origin rpy="0 0 0" xyz="-3.8 0.7 0.285"/>
       <parent link="${namespace}/base_link"/>
       <child link="left_engine_link"/>
@@ -31,5 +38,5 @@
     <joint name="left_engine_propeller_joint" type="continuous">
       <axis rpy="0 0 0" xyz="1 0 0"/>
-      <origin xyz="0 0 0" rpy="0 0 0"/>
+      <origin xyz="0.1 0 -0.191" rpy="0 0 0"/>
       <parent link="left_engine_link"/>
       <child link="left_propeller_link"/>
@@ -39,4 +46,10 @@
     <!-- Dummy link, which usv_gazebo_thrust_plugin looks for -->
     <link name="right_engine_link">
+      <visual>
+        <origin rpy="0 0 -${pi/2}" xyz="0 0 0"/>
+        <geometry>
+          <mesh filename="package://sandwich_description/models/thruster/thruster.dae" scale="4 4 4"/>
+        </geometry>
+      </visual>
       <inertial>
         <mass value="0.1"/>
@@ -47,6 +60,7 @@
     <link name="right_propeller_link">
       <visual>
+        <origin rpy="0 0 -${pi/2}" xyz="0 0 0"/>
         <geometry>
-          <mesh filename="package://sandwich_description/models/propeller/propeller.dae"/>
+          <mesh filename="package://sandwich_description/models/propeller/propeller.dae" scale="4 4 4"/>
         </geometry>
       </visual>
@@ -58,6 +72,6 @@
     <!-- Dummy joint, which usv_gazebo_thrust_plugin looks for -->
     <joint name="right_chasis_engine_joint" type="revolute">
-      <axis xyz="0 0 1"/>
-      <origin rpy="0 0 0" xyz="-6.103 -0.911 0.016"/>
+      <axis xyz="1 0 0"/>
+      <origin rpy="0 0 0" xyz="-3.8 -0.7 0.285"/>
       <parent link="${namespace}/base_link"/>
       <child link="right_engine_link"/>
@@ -66,5 +80,5 @@
     <joint name="right_engine_propeller_joint" type="continuous">
       <axis rpy="0 0 0" xyz="1 0 0"/>
-      <origin xyz="0 0 0" rpy="0 0 0"/>
+      <origin xyz="0.1 0 -0.191" rpy="0 0 0"/>
       <parent link="right_engine_link"/>
       <child link="right_propeller_link"/>
