Commit message: Modify thrusters to provide realistic behavior

File: sandwich_description/urdf/sandwich_thruster_config.xacro (robot description, xacro)
@@ -13,6 +13,6 @@
 			<mappingType>0</mappingType>
 			<maxCmd>1.0</maxCmd>
-			<maxForceFwd>12000.0</maxForceFwd>
-			<maxForceRev>-5000.0</maxForceRev>
+			<maxForceFwd>50000.0</maxForceFwd>
+			<maxForceRev>-50000.0</maxForceRev>
 			<maxAngle>${pi/2}</maxAngle>
 		</thruster>

File: sandwich_description/urdf/thrusters.xacro (robot description, xacro)
@@ -31,5 +31,5 @@
     <joint name="left_chasis_engine_joint" type="revolute">
       <axis xyz="1 0 0"/>
-      <origin rpy="0 0 0" xyz="-3.8 0.7 0.285"/>
+      <origin rpy="0 0 0" xyz="-3.8 1.2 0.285"/>
       <parent link="${namespace}/base_link"/>
       <child link="left_engine_link"/>
@@ -73,5 +73,5 @@
     <joint name="right_chasis_engine_joint" type="revolute">
       <axis xyz="1 0 0"/>
-      <origin rpy="0 0 0" xyz="-3.8 -0.7 0.285"/>
+      <origin rpy="0 0 0" xyz="-3.8 -1.2 0.285"/>
       <parent link="${namespace}/base_link"/>
       <child link="right_engine_link"/>
